Commit message: CP2: Fix mesh paths and xacro includes for ROS2

File: src/spyderr_description/urdf/spyderr.xacro (robot description, xacro)
@@ -1,7 +1,10 @@
 <?xml version="1.0" ?>
 <robot name="spyderr" xmlns:xacro="http://www.ros.org/wiki/xacro">
-<xacro:include filename="$(find spyderr_description)/urdf/materials.xacro" />
-<xacro:include filename="$(find spyderr_description)/urdf/spyderr.ros2control" />
-<xacro:include filename="$(find spyderr_description)/urdf/spyderr.gazebo" />
+<!-- ROS 2–safe package share root -->
+<xacro:property name="pkg_share" value="$(find spyderr_description)"/>
+<xacro:property name="mesh_dir"  value="${pkg_share}/meshes"/>
+<xacro:include filename="${pkg_share}/urdf/materials.xacro" />
+<xacro:include filename="${pkg_share}/urdf/spyderr.ros2control" />
+<xacro:include filename="${pkg_share}/urdf/spyderr.gazebo" />
 <link name="base_link">
   <inertial>
@@ -13,5 +16,5 @@
     <origin xyz="0 0 0" rpy="0 0 0"/>
     <geometry>
-      <mesh filename="file://$(find spyderr_description)/meshes/base_link.stl" scale="0.001 0.001 0.001"/>
+      <mesh filename="file://${mesh_dir}/base_link.stl" scale="0.001 0.001 0.001"/>
     </geometry>
     <material name="silver"/>
@@ -20,5 +23,5 @@
     <origin xyz="0 0 0" rpy="0 0 0"/>
     <geometry>
-      <mesh filename="file://$(find spyderr_description)/meshes/base_link.stl" scale="0.001 0.001 0.001"/>
+      <mesh filename="file://${mesh_dir}/base_link.stl" scale="0.001 0.001 0.001"/>
     </geometry>
   </collision>
@@ -33,5 +36,5 @@
     <origin xyz="0.0749 -0.0542 -0.0528" rpy="0 0 0"/>
     <geometry>
-      <mesh filename="file://$(find spyderr_description)/meshes/coxa_FR_1.stl" scale="0.001 0.001 0.001"/>
+      <mesh filename="file://${mesh_dir}/coxa_FR_1.stl" scale="0.001 0.001 0.001"/>
     </geometry>
     <material name="silver"/>
@@ -40,5 +43,5 @@
     <origin xyz="0.0749 -0.0542 -0.0528" rpy="0 0 0"/>
     <geometry>
-      <mesh filename="file://$(find spyderr_description)/meshes/coxa_FR_1.stl" scale="0.001 0.001 0.001"/>
+      <mesh filename="file://${mesh_dir}/coxa_FR_1.stl" scale="0.001 0.001 0.001"/>
     </geometry>
   </collision>
@@ -53,5 +56,5 @@
     <origin xyz="0.113987 -0.023232 -0.0627" rpy="0 0 0"/>
     <geometry>
-      <mesh filename="file://$(find spyderr_description)/meshes/femur_FR_1.stl" scale="0.001 0.001 0.001"/>
+      <mesh filename="file://${mesh_dir}/femur_FR_1.stl" scale="0.001 0.001 0.001"/>
     </geometry>
     <material name="silver"/>
@@ -60,5 +63,5 @@
     <origin xyz="0.113987 -0.023232 -0.0627" rpy="0 0 0"/>
     <geometry>
-      <mesh filename="file://$(find spyderr_description)/meshes/femur_FR_1.stl" scale="0.001 0.001 0.001"/>
+      <mesh filename="file://${mesh_dir}/femur_FR_1.stl" scale="0.001 0.001 0.001"/>
     </geometry>
   </collision>
@@ -73,5 +76,5 @@
     <origin xyz="0.23362 -0.186207 0.144115" rpy="0 0 0"/>
     <geometry>
-      <mesh filename="file://$(find spyderr_description)/meshes/tibia_FR_1.stl" scale="0.001 0.001 0.001"/>
+      <mesh filename="file://${mesh_dir}/tibia_FR_1.stl" scale="0.001 0.001 0.001"/>
     </geometry>
     <material name="silver"/>
@@ -80,5 +83,5 @@
     <origin xyz="0.23362 -0.186207 0.144115" rpy="0 0 0"/>
     <geometry>
-      <mesh filename="file://$(find spyderr_description)/meshes/tibia_FR_1.stl" scale="0.001 0.001 0.001"/>
+      <mesh filename="file://${mesh_dir}/tibia_FR_1.stl" scale="0.001 0.001 0.001"/>
     </geometry>
   </collision>
@@ -93,5 +96,5 @@
     <origin xyz="-0.0549 -0.0542 -0.0528" rpy="0 0 0"/>
     <geometry>
-      <mesh filename="file://$(find spyderr_description)/meshes/coxa_BR_1.stl" scale="0.001 0.001 0.001"/>
+      <mesh filename="file://${mesh_dir}/coxa_BR_1.stl" scale="0.001 0.001 0.001"/>
     </geometry>
     <material name="silver"/>
@@ -100,5 +103,5 @@
     <origin xyz="-0.0549 -0.0542 -0.0528" rpy="0 0 0"/>
     <geometry>
-      <mesh filename="file://$(find spyderr_description)/meshes/coxa_BR_1.stl" scale="0.001 0.001 0.001"/>
+      <mesh filename="file://${mesh_dir}/coxa_BR_1.stl" scale="0.001 0.001 0.001"/>
     </geometry>
   </collision>
@@ -113,5 +116,5 @@
     <origin xyz="-0.193264 0.021095 -0.0627" rpy="0 0 0"/>
     <geometry>
-      <mesh filename="file://$(find spyderr_description)/meshes/femur_BR_1.stl" scale="0.001 0.001 0.001"/>
+      <mesh filename="file://${mesh_dir}/femur_BR_1.stl" scale="0.001 0.001 0.001"/>
     </geometry>
     <material name="silver"/>
@@ -120,5 +123,5 @@
     <origin xyz="-0.193264 0.021095 -0.0627" rpy="0 0 0"/>
     <geometry>
-      <mesh filename="file://$(find spyderr_description)/meshes/femur_BR_1.stl" scale="0.001 0.001 0.001"/>
+      <mesh filename="file://${mesh_dir}/femur_BR_1.stl" scale="0.001 0.001 0.001"/>
     </geometry>
   </collision>
@@ -133,5 +136,5 @@
     <origin xyz="-0.218025 -0.244252 -0.156756" rpy="0 0 0"/>
     <geometry>
-      <mesh filename="file://$(find spyderr_description)/meshes/tibia_BR_1.stl" scale="0.001 0.001 0.001"/>
+      <mesh filename="file://${mesh_dir}/tibia_BR_1.stl" scale="0.001 0.001 0.001"/>
     </geometry>
     <material name="silver"/>
@@ -140,5 +143,5 @@
     <origin xyz="-0.218025 -0.244252 -0.156756" rpy="0 0 0"/>
     <geometry>
-      <mesh filename="file://$(find spyderr_description)/meshes/tibia_BR_1.stl" scale="0.001 0.001 0.001"/>
+      <mesh filename="file://${mesh_dir}/tibia_BR_1.stl" scale="0.001 0.001 0.001"/>
     </geometry>
   </collision>
@@ -153,5 +156,5 @@
     <origin xyz="0.0749 0.0942 -0.0528" rpy="0 0 0"/>
     <geometry>
-      <mesh filename="file://$(find spyderr_description)/meshes/coxa_FL_1.stl" scale="0.001 0.001 0.001"/>
+      <mesh filename="file://${mesh_dir}/coxa_FL_1.stl" scale="0.001 0.001 0.001"/>
     </geometry>
     <material name="silver"/>
@@ -160,5 +163,5 @@
     <origin xyz="0.0749 0.0942 -0.0528" rpy="0 0 0"/>
     <geometry>
-      <mesh filename="file://$(find spyderr_description)/meshes/coxa_FL_1.stl" scale="0.001 0.001 0.001"/>
+      <mesh filename="file://${mesh_dir}/coxa_FL_1.stl" scale="0.001 0.001 0.001"/>
     </geometry>
   </collision>
@@ -173,5 +176,5 @@
     <origin xyz="-0.084253 -0.049848 -0.0627" rpy="0 0 0"/>
     <geometry>
-      <mesh filename="file://$(find spyderr_description)/meshes/femur_FL_1.stl" scale="0.001 0.001 0.001"/>
+      <mesh filename="file://${mesh_dir}/femur_FL_1.stl" scale="0.001 0.001 0.001"/>
     </geometry>
     <material name="silver"/>
@@ -180,5 +183,5 @@
     <origin xyz="-0.084253 -0.049848 -0.0627" rpy="0 0 0"/>
     <geometry>
-      <mesh filename="file://$(find spyderr_description)/meshes/femur_FL_1.stl" scale="0.001 0.001 0.001"/>
+      <mesh filename="file://${mesh_dir}/femur_FL_1.stl" scale="0.001 0.001 0.001"/>
     </geometry>
   </collision>
@@ -193,5 +196,5 @@
     <origin xyz="-0.017251 0.028976 0.099956" rpy="0 0 0"/>
     <geometry>
-      <mesh filename="file://$(find spyderr_description)/meshes/tibia_FL_1.stl" scale="0.001 0.001 0.001"/>
+      <mesh filename="file://${mesh_dir}/tibia_FL_1.stl" scale="0.001 0.001 0.001"/>
     </geometry>
     <material name="silver"/>
@@ -200,5 +203,5 @@
     <origin xyz="-0.017251 0.028976 0.099956" rpy="0 0 0"/>
     <geometry>
-      <mesh filename="file://$(find spyderr_description)/meshes/tibia_FL_1.stl" scale="0.001 0.001 0.001"/>
+      <mesh filename="file://${mesh_dir}/tibia_FL_1.stl" scale="0.001 0.001 0.001"/>
     </geometry>
   </collision>
@@ -213,5 +216,5 @@
     <origin xyz="-0.0549 0.0942 -0.0528" rpy="0 0 0"/>
     <geometry>
-      <mesh filename="file://$(find spyderr_description)/meshes/coxa_BL_1.stl" scale="0.001 0.001 0.001"/>
+      <mesh filename="file://${mesh_dir}/coxa_BL_1.stl" scale="0.001 0.001 0.001"/>
     </geometry>
     <material name="silver"/>
@@ -220,5 +223,5 @@
     <origin xyz="-0.0549 0.0942 -0.0528" rpy="0 0 0"/>
     <geometry>
-      <mesh filename="file://$(find spyderr_description)/meshes/coxa_BL_1.stl" scale="0.001 0.001 0.001"/>
+      <mesh filename="file://${mesh_dir}/coxa_BL_1.stl" scale="0.001 0.001 0.001"/>
     </geometry>
   </collision>
@@ -233,5 +236,5 @@
     <origin xyz="0.203531 0.10503 -0.0627" rpy="0 0 0"/>
     <geometry>
-      <mesh filename="file://$(find spyderr_description)/meshes/femur_BL_1.stl" scale="0.001 0.001 0.001"/>
+      <mesh filename="file://${mesh_dir}/femur_BL_1.stl" scale="0.001 0.001 0.001"/>
     </geometry>
     <material name="silver"/>
@@ -240,5 +243,5 @@
     <origin xyz="0.203531 0.10503 -0.0627" rpy="0 0 0"/>
     <geometry>
-      <mesh filename="file://$(find spyderr_description)/meshes/femur_BL_1.stl" scale="0.001 0.001 0.001"/>
+      <mesh filename="file://${mesh_dir}/femur_BL_1.stl" scale="0.001 0.001 0.001"/>
     </geometry>
   </collision>
@@ -253,5 +256,5 @@
     <origin xyz="-0.021579 0.033246 -0.201375" rpy="0 0 0"/>
     <geometry>
-      <mesh filename="file://$(find spyderr_description)/meshes/tibia_BL_1.stl" scale="0.001 0.001 0.001"/>
+      <mesh filename="file://${mesh_dir}/tibia_BL_1.stl" scale="0.001 0.001 0.001"/>
     </geometry>
     <material name="silver"/>
@@ -260,5 +263,5 @@
     <origin xyz="-0.021579 0.033246 -0.201375" rpy="0 0 0"/>
     <geometry>
-      <mesh filename="file://$(find spyderr_description)/meshes/tibia_BL_1.stl" scale="0.001 0.001 0.001"/>
+      <mesh filename="file://${mesh_dir}/tibia_BL_1.stl" scale="0.001 0.001 0.001"/>
     </geometry>
   </collision>
@@ -273,5 +276,5 @@
     <origin xyz="-0.064 0.02 -0.0877" rpy="0 0 0"/>
     <geometry>
-      <mesh filename="file://$(find spyderr_description)/meshes/camera_stand_1.stl" scale="0.001 0.001 0.001"/>
+      <mesh filename="file://${mesh_dir}/camera_stand_1.stl" scale="0.001 0.001 0.001"/>
     </geometry>
     <material name="silver"/>
@@ -280,5 +283,5 @@
     <origin xyz="-0.064 0.02 -0.0877" rpy="0 0 0"/>
     <geometry>
-      <mesh filename="file://$(find spyderr_description)/meshes/camera_stand_1.stl" scale="0.001 0.001 0.001"/>
+      <mesh filename="file://${mesh_dir}/camera_stand_1.stl" scale="0.001 0.001 0.001"/>
     </geometry>
   </collision>
@@ -293,5 +296,5 @@
     <origin xyz="-0.061225 0.026 -0.1647" rpy="0 0 0"/>
     <geometry>
-      <mesh filename="file://$(find spyderr_description)/meshes/camera_1.stl" scale="0.001 0.001 0.001"/>
+      <mesh filename="file://${mesh_dir}/camera_1.stl" scale="0.001 0.001 0.001"/>
     </geometry>
     <material name="silver"/>
@@ -300,5 +303,5 @@
     <origin xyz="-0.061225 0.026 -0.1647" rpy="0 0 0"/>
     <geometry>
-      <mesh filename="file://$(find spyderr_description)/meshes/camera_1.stl" scale="0.001 0.001 0.001"/>
+      <mesh filename="file://${mesh_dir}/camera_1.stl" scale="0.001 0.001 0.001"/>
     </geometry>
   </collision>
@@ -313,5 +316,5 @@
     <origin xyz="0.069407 0.019459 -0.0877" rpy="0 0 0"/>
     <geometry>
-      <mesh filename="file://$(find spyderr_description)/meshes/lidar_1.stl" scale="0.001 0.001 0.001"/>
+      <mesh filename="file://${mesh_dir}/lidar_1.stl" scale="0.001 0.001 0.001"/>
     </geometry>
     <material name="silver"/>
@@ -320,5 +323,5 @@
     <origin xyz="0.069407 0.019459 -0.0877" rpy="0 0 0"/>
     <geometry>
-      <mesh filename="file://$(find spyderr_description)/meshes/lidar_1.stl" scale="0.001 0.001 0.001"/>
+      <mesh filename="file://${mesh_dir}/lidar_1.stl" scale="0.001 0.001 0.001"/>
     </geometry>
   </collision>
@@ -333,5 +336,5 @@
     <origin xyz="-0.01 0.02 -0.0877" rpy="0 0 0"/>
     <geometry>
-      <mesh filename="file://$(find spyderr_description)/meshes/imu_1.stl" scale="0.001 0.001 0.001"/>
+      <mesh filename="file://${mesh_dir}/imu_1.stl" scale="0.001 0.001 0.001"/>
     </geometry>
     <material name="silver"/>
@@ -340,5 +343,5 @@
     <origin xyz="-0.01 0.02 -0.0877" rpy="0 0 0"/>
     <geometry>
-      <mesh filename="file://$(find spyderr_description)/meshes/imu_1.stl" scale="0.001 0.001 0.001"/>
+      <mesh filename="file://${mesh_dir}/imu_1.stl" scale="0.001 0.001 0.001"/>
     </geometry>
   </collision>

Commit message: cp3: deterministic link-local meshes for visuals + ament_python install fix

File: src/spyderr_description/urdf/spyderr.xacro (robot description, xacro)
@@ -34,7 +34,7 @@
   </inertial>
   <visual>
-    <origin xyz="0.0749 -0.0542 -0.0528" rpy="0 0 0"/>
-    <geometry>
-      <mesh filename="file://${mesh_dir}/coxa_FR_1.stl" scale="0.001 0.001 0.001"/>
+    <origin xyz="0 0 0" rpy="0 0 0"/>
+    <geometry>
+      <mesh filename="file://${mesh_dir}/link_local/coxa_FR_1__visual0.stl" scale="0.001 0.001 0.001"/>
     </geometry>
     <material name="silver"/>
@@ -54,7 +54,7 @@
   </inertial>
   <visual>
-    <origin xyz="0.113987 -0.023232 -0.0627" rpy="0 0 0"/>
-    <geometry>
-      <mesh filename="file://${mesh_dir}/femur_FR_1.stl" scale="0.001 0.001 0.001"/>
+    <origin xyz="0 0 0" rpy="0 0 0"/>
+    <geometry>
+      <mesh filename="file://${mesh_dir}/link_local/femur_FR_1__visual0.stl" scale="0.001 0.001 0.001"/>
     </geometry>
     <material name="silver"/>
@@ -74,7 +74,7 @@
   </inertial>
   <visual>
-    <origin xyz="0.23362 -0.186207 0.144115" rpy="0 0 0"/>
-    <geometry>
-      <mesh filename="file://${mesh_dir}/tibia_FR_1.stl" scale="0.001 0.001 0.001"/>
+    <origin xyz="0 0 0" rpy="0 0 0"/>
+    <geometry>
+      <mesh filename="file://${mesh_dir}/link_local/tibia_FR_1__visual0.stl" scale="0.001 0.001 0.001"/>
     </geometry>
     <material name="silver"/>
@@ -94,7 +94,7 @@
   </inertial>
   <visual>
-    <origin xyz="-0.0549 -0.0542 -0.0528" rpy="0 0 0"/>
-    <geometry>
-      <mesh filename="file://${mesh_dir}/coxa_BR_1.stl" scale="0.001 0.001 0.001"/>
+    <origin xyz="0 0 0" rpy="0 0 0"/>
+    <geometry>
+      <mesh filename="file://${mesh_dir}/link_local/coxa_BR_1__visual0.stl" scale="0.001 0.001 0.001"/>
     </geometry>
     <material name="silver"/>
@@ -114,7 +114,7 @@
   </inertial>
   <visual>
-    <origin xyz="-0.193264 0.021095 -0.0627" rpy="0 0 0"/>
-    <geometry>
-      <mesh filename="file://${mesh_dir}/femur_BR_1.stl" scale="0.001 0.001 0.001"/>
+    <origin xyz="0 0 0" rpy="0 0 0"/>
+    <geometry>
+      <mesh filename="file://${mesh_dir}/link_local/femur_BR_1__visual0.stl" scale="0.001 0.001 0.001"/>
     </geometry>
     <material name="silver"/>
@@ -134,7 +134,7 @@
   </inertial>
   <visual>
-    <origin xyz="-0.218025 -0.244252 -0.156756" rpy="0 0 0"/>
-    <geometry>
-      <mesh filename="file://${mesh_dir}/tibia_BR_1.stl" scale="0.001 0.001 0.001"/>
+    <origin xyz="0 0 0" rpy="0 0 0"/>
+    <geometry>
+      <mesh filename="file://${mesh_dir}/link_local/tibia_BR_1__visual0.stl" scale="0.001 0.001 0.001"/>
     </geometry>
     <material name="silver"/>
@@ -154,7 +154,7 @@
   </inertial>
   <visual>
-    <origin xyz="0.0749 0.0942 -0.0528" rpy="0 0 0"/>
-    <geometry>
-      <mesh filename="file://${mesh_dir}/coxa_FL_1.stl" scale="0.001 0.001 0.001"/>
+    <origin xyz="0 0 0" rpy="0 0 0"/>
+    <geometry>
+      <mesh filename="file://${mesh_dir}/link_local/coxa_FL_1__visual0.stl" scale="0.001 0.001 0.001"/>
     </geometry>
     <material name="silver"/>
@@ -174,7 +174,7 @@
   </inertial>
   <visual>
-    <origin xyz="-0.084253 -0.049848 -0.0627" rpy="0 0 0"/>
-    <geometry>
-      <mesh filename="file://${mesh_dir}/femur_FL_1.stl" scale="0.001 0.001 0.001"/>
+    <origin xyz="0 0 0" rpy="0 0 0"/>
+    <geometry>
+      <mesh filename="file://${mesh_dir}/link_local/femur_FL_1__visual0.stl" scale="0.001 0.001 0.001"/>
     </geometry>
     <material name="silver"/>
@@ -194,7 +194,7 @@
   </inertial>
   <visual>
-    <origin xyz="-0.017251 0.028976 0.099956" rpy="0 0 0"/>
-    <geometry>
-      <mesh filename="file://${mesh_dir}/tibia_FL_1.stl" scale="0.001 0.001 0.001"/>
+    <origin xyz="0 0 0" rpy="0 0 0"/>
+    <geometry>
+      <mesh filename="file://${mesh_dir}/link_local/tibia_FL_1__visual0.stl" scale="0.001 0.001 0.001"/>
     </geometry>
     <material name="silver"/>
@@ -214,7 +214,7 @@
   </inertial>
   <visual>
-    <origin xyz="-0.0549 0.0942 -0.0528" rpy="0 0 0"/>
-    <geometry>
-      <mesh filename="file://${mesh_dir}/coxa_BL_1.stl" scale="0.001 0.001 0.001"/>
+    <origin xyz="0 0 0" rpy="0 0 0"/>
+    <geometry>
+      <mesh filename="file://${mesh_dir}/link_local/coxa_BL_1__visual0.stl" scale="0.001 0.001 0.001"/>
     </geometry>
     <material name="silver"/>
@@ -234,7 +234,7 @@
   </inertial>
   <visual>
-    <origin xyz="0.203531 0.10503 -0.0627" rpy="0 0 0"/>
-    <geometry>
-      <mesh filename="file://${mesh_dir}/femur_BL_1.stl" scale="0.001 0.001 0.001"/>
+    <origin xyz="0 0 0" rpy="0 0 0"/>
+    <geometry>
+      <mesh filename="file://${mesh_dir}/link_local/femur_BL_1__visual0.stl" scale="0.001 0.001 0.001"/>
     </geometry>
     <material name="silver"/>
@@ -254,7 +254,7 @@
   </inertial>
   <visual>
-    <origin xyz="-0.021579 0.033246 -0.201375" rpy="0 0 0"/>
-    <geometry>
-      <mesh filename="file://${mesh_dir}/tibia_BL_1.stl" scale="0.001 0.001 0.001"/>
+    <origin xyz="0 0 0" rpy="0 0 0"/>
+    <geometry>
+      <mesh filename="file://${mesh_dir}/link_local/tibia_BL_1__visual0.stl" scale="0.001 0.001 0.001"/>
     </geometry>
     <material name="silver"/>
@@ -274,7 +274,7 @@
   </inertial>
   <visual>
-    <origin xyz="-0.064 0.02 -0.0877" rpy="0 0 0"/>
-    <geometry>
-      <mesh filename="file://${mesh_dir}/camera_stand_1.stl" scale="0.001 0.001 0.001"/>
+    <origin xyz="0 0 0" rpy="0 0 0"/>
+    <geometry>
+      <mesh filename="file://${mesh_dir}/link_local/camera_stand_1__visual0.stl" scale="0.001 0.001 0.001"/>
     </geometry>
     <material name="silver"/>
@@ -294,7 +294,7 @@
   </inertial>
   <visual>
-    <origin xyz="-0.061225 0.026 -0.1647" rpy="0 0 0"/>
-    <geometry>
-      <mesh filename="file://${mesh_dir}/camera_1.stl" scale="0.001 0.001 0.001"/>
+    <origin xyz="0 0 0" rpy="0 0 0"/>
+    <geometry>
+      <mesh filename="file://${mesh_dir}/link_local/camera_1__visual0.stl" scale="0.001 0.001 0.001"/>
     </geometry>
     <material name="silver"/>
@@ -314,7 +314,7 @@
   </inertial>
   <visual>
-    <origin xyz="0.069407 0.019459 -0.0877" rpy="0 0 0"/>
-    <geometry>
-      <mesh filename="file://${mesh_dir}/lidar_1.stl" scale="0.001 0.001 0.001"/>
+    <origin xyz="0 0 0" rpy="0 0 0"/>
+    <geometry>
+      <mesh filename="file://${mesh_dir}/link_local/lidar_1__visual0.stl" scale="0.001 0.001 0.001"/>
     </geometry>
     <material name="silver"/>
@@ -334,7 +334,7 @@
   </inertial>
   <visual>
-    <origin xyz="-0.01 0.02 -0.0877" rpy="0 0 0"/>
-    <geometry>
-      <mesh filename="file://${mesh_dir}/imu_1.stl" scale="0.001 0.001 0.001"/>
+    <origin xyz="0 0 0" rpy="0 0 0"/>
+    <geometry>
+      <mesh filename="file://${mesh_dir}/link_local/imu_1__visual0.stl" scale="0.001 0.001 0.001"/>
     </geometry>
     <material name="silver"/>
